File: kicad6/hellen1-mcu.kicad_pcb (KiCad board)
At the start: 2 copper layers, 46.5 x 37.4 mm, 92 parts, among them J101 TC2030-IDC-NL, J102 Net Tie, M101 Module:mcu/0.1, U101 AMS1117-3.3, U102 LMV324IPWR, U103 AP2337SA-7, U104 LMV324IPWR, U105 STM32F427IGT6, U106 LMV324IPWR, U107 LMV324IPWR, U108 LMV324IPWR, U109 LMV324IPWR, U111 XC6206P332MR, Y101 32.768 kHz, Y102 8.0 MHz

Commit message: update mcu-0.3 kicad-imported source
Parts:
- C101, C102, C103, C104, C105, C106, C107, C108, C109, C110, C111, C112, C113, C114, C115, C116, C117, C118, C119, C120, C121, C122, C123, C124, C125, C126, C127, C128, C129, C130, C131, C132, C135, C136, C137, C138, C139, C140: footprint General.pcblib:Cap -> General.pcblib:C0603
- D101, D107: footprint General.pcblib:D Schottky -> General.pcblib:SOD-123
- D102: footprint Small.PcbLib:D TVS Array 4 -> Small.PcbLib:SOT-26
- D103: value LED-RED -> LED-RED-0603; footprint General.pcblib:LED -> General.pcblib:LED-0603
- D104: value LED-GREEN -> LED-GREEN-0603; footprint General.pcblib:LED -> General.pcblib:LED-0603
- D105: value LED-BLUE -> LED-BLUE-0603; footprint General.pcblib:LED -> General.pcblib:LED-0603
- D106: value LED-YELLOW -> LED-YELLOW-0603; footprint General.pcblib:LED -> General.pcblib:LED-0603
- J101: footprint TH.PcbLib:JTAG-TC2030-IDC -> TH.PcbLib:JTAG-TC2030-IDC-NL
- J102: footprint General.pcblib:Net Tie -> General.pcblib:NET-TIE
- L101: footprint General.pcblib:Inductor -> General.pcblib:L0805
- M101: value Module:mcu/0.1 -> Module:mcu/0.3; footprint Mod.PcbLib:Mod-Hellen-MCU -> Mod.PcbLib:MOD_HELLEN_MCU
- R101, R107, R108, R109, R110, R112, R113, R117, R125: value 4k7 -> 4.7k; footprint Small.PcbLib:Res Array 4 -> Small.PcbLib:R0603_X4
- R102, R103, R104, R105, R106, R114, R116, R119, R120, R121, R124, R127, R128: footprint General.pcblib:Res -> General.pcblib:R0603
- R111, R115, R118, R126: value 4k7 -> 4.7k; footprint Small.PcbLib:Res Array 4 -> Small.PcbLib:R0603_x4
- R122, R123: value 10k -> 2.2k; footprint General.pcblib:Res -> General.pcblib:R0603
- R129, R130: footprint Small.PcbLib:Res Array 4 -> Small.PcbLib:R0603_x4
- R131: footprint General.pcblib:Res -> General.pcblib:R0402
- U101: footprint Small.PcbLib:78xx -> Small.PcbLib:SOT-223
- U102, U104, U106, U107, U108, U109: footprint IC.PcbLib:MCP6004 -> IC.PcbLib:TSSOP14
- U103, U111: footprint Small.PcbLib:78xx -> Small.PcbLib:SOT-23
- U105: footprint IC.PcbLib:STM32H743Ix -> IC.PcbLib:LQFP176
- Y101: footprint Small.PcbLib:Quartz -> Small.PcbLib:QUARTZ-SMD2012
- Y102: footprint Small.PcbLib:Quartz -> Small.PcbLib:QUARTZ-SMD5032
Connections:
- net SPI_SD_CS renamed SPI2_CS
- net SPI_SD_MISO renamed SPI2_MISO
- net SPI_SD_MOSI renamed SPI2_MOSI
- net SPI_SD_SCK renamed SPI2_SCK
- M101 pad E10: OUT_IO5 -> OUT_IO10
- M101 pad E11: OUT_IO6 -> OUT_IO9
- M101 pad E12: OUT_IO7 -> OUT_IO2
- M101 pad E13: OUT_IO8 -> OUT_IO12
- M101 pad E14: OUT_PWM1 -> OUT_PWM2
- M101 pad E15: OUT_PWM2 -> OUT_PWM3
- M101 pad E16: OUT_PWM3 -> OUT_PWM4
- M101 pad E17: OUT_PWM4 -> OUT_PWM5
- M101 pad E18: OUT_PWM5 -> OUT_PWM6
- M101 pad E19: OUT_PWM6 -> OUT_PWM7
- M101 pad E20: OUT_IO9 -> OUT_IO11
- M101 pad E21: OUT_IO10 -> OUT_IO7
- M101 pad E22: OUT_IO11 -> OUT_IO8
- M101 pad E23: OUT_IO12 -> OUT_IO4
- M101 pad E27: OUT_PWM7 -> OUT_PWM1
- M101 pad E6: OUT_IO1 -> OUT_IO3
- M101 pad E7: OUT_IO2 -> OUT_IO5
- M101 pad E8: OUT_IO3 -> OUT_IO1
- M101 pad E9: OUT_IO4 -> OUT_IO6
- U105 pad 101: OUT_PWM7 -> OUT_PWM1
- U105 pad 104: OUT_PWM5 -> OUT_PWM6
- U105 pad 105: OUT_PWM6 -> OUT_PWM7
- U105 pad 106: OUT_IO9 -> OUT_IO11
- U105 pad 107: OUT_IO10 -> OUT_IO7
- U105 pad 108: OUT_IO11 -> OUT_IO8
- U105 pad 109: OUT_IO12 -> OUT_IO4
- U105 pad 115: OUT_PWM1 -> OUT_PWM2
- U105 pad 116: OUT_PWM2 -> OUT_PWM3
- U105 pad 117: OUT_PWM3 -> OUT_PWM4
- U105 pad 118: OUT_PWM4 -> OUT_PWM5
- U105 pad 119: OUT_IO8 -> OUT_IO12
- U105 pad 120: OUT_IO7 -> OUT_IO2
- U105 pad 128: OUT_IO2 -> OUT_IO5
- U105 pad 129: OUT_IO3 -> OUT_IO1
- U105 pad 130: OUT_IO4 -> OUT_IO6
- U105 pad 131: OUT_IO5 -> OUT_IO10
- U105 pad 132: OUT_IO6 -> OUT_IO9
- U105 pad 133: OUT_IO1 -> OUT_IO3
- U105 pad 144: (no net) -> IO5
- U105 pad 146: IO5 -> (no net)
Routing:
- net OUT_IO9: track 15.7 -> 30.8 mm
- net OUT_IO3: track 20.5 -> 34.7 mm
- net OUT_IO1: track 34.7 -> 20.5 mm
- net OUT_PWM5: track 12.0 -> 25.4 mm
- net OUT_IO10: track 17.5 -> 25.6 mm
- net OUT_IO5: track 25.6 -> 18.0 mm
- net OUT_IO6: track 30.8 -> 24.3 mm
- net OUT_PWM4: track 25.4 -> 20.0 mm
- net OUT_PWM1: track 15.5 -> 10.5 mm
- net OUT_IO7: track 21.5 -> 17.5 mm
- net OUT_IO4: track 24.3 -> 20.6 mm
- net OUT_IO2: track 18.0 -> 21.5 mm
- net OUT_IO8: track 22.6 -> 19.1 mm
- net OUT_IO11: track 19.1 -> 15.7 mm
- net OUT_PWM7: track 10.5 -> 13.7 mm
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Other:
- board text added: "'.ItemAndRevision'"
