File: kicad6/hellen1-mcu.kicad_sch (KiCad schematic)
At the start: 92 parts, among them J101 *

Commit message: move kicad src files into a separate folder
Parts:
- C101, C105, C106, C107, C108, C109, C110, C111, C112, C113, C117, C118, C119, C120, C121, C122, C123, C124, C125, C126, C127, C128, C129, C130, C135, C139: value ~ -> 100n; Comment 100n -> (none)
- C102, C103, C104, C137, C138, C140: value ~ -> 4.7u; Comment 4.7u -> (none)
- C114, C131: value ~ -> 2.2u; Comment 2.2u -> (none)
- C115, C116: value ~ -> 12p; Comment 12p -> (none)
- C132, C136: value ~ -> 18p; Comment 18p -> (none)
- D101, D107: value ~ -> B5819W; Comment B5819W -> (none)
- D102: value ~ -> SRV05-4-P-T7; Comment SRV05-4-P-T7 -> (none)
- D103: value ~ -> LED-RED-0603; Comment LED-RED -> (none)
- D104: value ~ -> LED-GREEN-0603; Comment LED-GREEN -> (none)
- D105: value ~ -> LED-BLUE-0603; Comment LED-BLUE -> (none)
- D106: value ~ -> LED-YELLOW-0603; Comment LED-YELLOW -> (none)
- J101: value * -> TC2030-IDC-NL; Altium_Value (none) -> *; Comment TC2030-IDC-NL -> (none)
- J102: value ~ -> Net Tie; Comment Net Tie -> (none)
- L101: value =Comment -> SDFL2012Q3R3KTF; Altium_Value (none) -> ${VALUE}; Comment SDFL2012Q3R3KTF -> (none)
- M101: value ~ -> Module:mcu/0.1; Comment Module:mcu/0.1 -> (none)
- R101, R107, R108, R109, R110, R111, R112, R113, R115, R117, R118, R125, R126: value ~ -> 4.7k; Comment 4k7 -> (none)
- R102, R103, R105, R121, R122, R123, R127, R128, R129, R130: value ~ -> 10k; Comment 10k -> (none)
- R104, R106: value ~ -> 100; Comment 100 -> (none)
- R114: value ~ -> 47; Comment 47 -> (none)
- R116, R119, R120, R124: value ~ -> 510; Comment 510 -> (none)
- R131: value ~ -> 0; Comment 0 -> (none)
- U101: value ~ -> AMS1117-3.3; Comment AMS1117-3.3 -> (none)
- U102, U104, U106, U107, U108, U109: value ~ -> LMV324IPWR; Comment LMV324IPWR -> (none)
- U103: value ~ -> AP2337SA-7; Comment AP2337SA-7 -> (none)
- U105: value ~ -> STM32F427IGT6; Comment STM32F427IGT6 -> (none)
- U111: value ~ -> XC6206P332MR; Comment XC6206P332MR -> (none)
- Y101: value ~ -> 32.768 kHz; Comment 32.768 kHz -> (none)
- Y102: value ~ -> 8.0 MHz; Comment 8.0 MHz -> (none)
Connections:
- net BOOT0: now also R127.2
- net GND: now also R129.5, R129.6, R129.7, R130.5, R130.6, R130.7
- net IO5: now also M101.N12 (IO1), U105.144 (PD2); no longer M101.N12 (IO1), U105.146 (PD4)
- net IO6: now also M101.N13 (IO2); no longer M101.N13 (IO2)
- net IO7: now also M101.N14 (IO3); no longer M101.N14 (IO3)
- net IO8: now also M101.N15 (IO4); no longer M101.N15 (IO4)
- net OUT_IO1: now also M101.E8 (OUT_IO1), U105.129 (PH14); no longer M101.E6 (OUT_IO1), U105.133 (PI2)
- net OUT_IO10: now also M101.E10 (OUT_IO10), U105.131 (PI0); no longer M101.E21 (OUT_IO10), U105.107 (PG3)
- net OUT_IO11: now also M101.E20 (OUT_IO11), U105.106 (PG2); no longer M101.E22 (OUT_IO11), U105.108 (PG4)
- net OUT_IO12: now also M101.E13 (OUT_IO12), U105.119 (PA8); no longer M101.E23 (OUT_IO12), U105.109 (PG5)
- net OUT_IO2: now also M101.E12 (OUT_IO2), U105.120 (PA9); no longer M101.E7 (OUT_IO2), U105.128 (PH13)
- net OUT_IO3: now also M101.E6 (OUT_IO3), U105.133 (PI2); no longer M101.E8 (OUT_IO3), U105.129 (PH14)
- net OUT_IO4: now also M101.E23 (OUT_IO4), U105.109 (PG5); no longer M101.E9 (OUT_IO4), U105.130 (PH15)
- net OUT_IO5: now also M101.E7 (OUT_IO5), U105.128 (PH13); no longer M101.E10 (OUT_IO5), U105.131 (PI0)
- net OUT_IO6: now also M101.E9 (OUT_IO6), U105.130 (PH15); no longer M101.E11 (OUT_IO6), U105.132 (PI1)
- net OUT_IO7: now also M101.E21 (OUT_IO7), U105.107 (PG3); no longer M101.E12 (OUT_IO7), U105.120 (PA9)
- net OUT_IO8: now also M101.E22 (OUT_IO8), U105.108 (PG4); no longer M101.E13 (OUT_IO8), U105.119 (PA8)
- net OUT_IO9: now also M101.E11 (OUT_IO9), U105.132 (PI1); no longer M101.E20 (OUT_IO9), U105.106 (PG2)
- net OUT_PWM1: now also M101.E27 (OUT_PWM1), U105.101 (PD13); no longer M101.E14 (OUT_PWM1), U105.115 (PC6)
- net OUT_PWM2: now also M101.E14 (OUT_PWM2), U105.115 (PC6); no longer M101.E15 (OUT_PWM2), U105.116 (PC7)
- net OUT_PWM3: now also M101.E15 (OUT_PWM3), U105.116 (PC7); no longer M101.E16 (OUT_PWM3), U105.117 (PC8)
- net OUT_PWM4: now also M101.E16 (OUT_PWM4), U105.117 (PC8); no longer M101.E17 (OUT_PWM4), U105.118 (PC9)
- net OUT_PWM5: now also M101.E17 (OUT_PWM5), U105.118 (PC9); no longer M101.E18 (OUT_PWM5), U105.104 (PD14)
- net OUT_PWM6: now also M101.E18 (OUT_PWM6), U105.104 (PD14); no longer M101.E19 (OUT_PWM6), U105.105 (PD15)
- net OUT_PWM7: now also M101.E19 (OUT_PWM7), U105.105 (PD15); no longer M101.E27 (OUT_PWM7), U105.101 (PD13)
- net V33: now also D104.1 (A), D105.1 (A)
- net at C116.2: now also U105.10 (PC15/OSC32_OUT), Y101.2 (OSC2)
- net at R126.1, U109.9 (VinC-): now also U109.8 (VoutC)
- net at R126.4, U109.6 (VinB-): now also U109.7 (VoutB)
- net at R118.1, U109.2 (VinA-): now also U109.1 (VoutA)
- net at R118.4, U109.13 (VinD-): now also U109.14 (VoutD)
- net at U102.1 (VoutA): now also R101.1, U102.2 (VinA-)
- net at R101.4, U102.13 (VinD-): now also U102.14 (VoutD)
- net at R107.1, U102.6 (VinB-): now also U102.7 (VoutB)
- net at U102.8 (VoutC): now also R107.4, U102.9 (VinC-)
- net at R117.1, U108.9 (VinC-): now also U108.8 (VoutC)
- net at R113.1, U108.2 (VinA-): now also U108.1 (VoutA)
- net at U104.1 (VoutA): now also R108.1, U104.2 (VinA-)
- net at U104.8 (VoutC): now also R109.1, U104.9 (VinC-)
- net at U107.1 (VoutA): now also R111.1, U107.2 (VinA-)
- net at R111.4, U107.13 (VinD-): now also U107.14 (VoutD)
- net at R115.4, U107.6 (VinB-): now also U107.7 (VoutB)
- net at U107.8 (VoutC): now also R115.1, U107.9 (VinC-)
- net at R110.1, U106.2 (VinA-): now also U106.1 (VoutA)
- net at R112.1, U106.9 (VinC-): now also U106.8 (VoutC)
- net SPI_SD_CS renamed SPI2_CS
- net SPI_SD_MISO renamed SPI2_MISO
- net SPI_SD_MOSI renamed SPI2_MOSI
- net SPI_SD_SCK renamed SPI2_SCK

Commit message: update mcu-0.3 kicad-imported source
Parts:
- M101: value Module:mcu/0.1 -> Module:mcu/0.3
- R122, R123: value 10k -> 2.2k; Supplier Part Number 3 C25804 -> C4190
