File: hellen72_NB2.kicad_sch (KiCad schematic)
At the start: 185 parts, among them J1 USB_B_Mini, J11 Conn_01x01, J13 Conn_01x01, J14 Conn_01x01, J15 Conn_01x01, J16 Conn_01x01, J17 Conn_01x01, J19 Conn_01x01, J2 Conn_01x05_Male, J20 Conn_01x01, J21 Conn_01x01, J22 Conn_01x01, J24 Conn_01x01, J25 AudioJack3_SwitchTR, J27 Conn_01x06, J3 MiniFit, J4 Conn_02x12_Odd_Even, J5 USB_B, J6 ETB, M1 Module-input-0.1, M10 Module-power12-0.2, M11 Module-power5-0.2, M12 Module-wbo-0.3, M13 Module-can-0.1, M2 Module-ign8-0.1, M3 Module-mcu144-0.5, M4 Module-sd-0.1, M5 Module-output-0.3, M6 Module-dinput4-0.1, M7 Module-stlink-0.1, M8 Module-can-0.1, M9 Module-knock-0.1, P1 Pad, P10 Pad, P11 Pad, P12 Pad, P13 Pad, P14 Pad, P15 Pad, P16 Pad, P17 Pad, P18 Pad, P19 Pad, P2 1123794-2, P20 Pad, P22 Pad, P23 Pad, P28 Pad, P3 Pad, P38 Pad, P4 Pad, P44 Pad, P48 Pad, P49 Pad, P5 Pad, P50 Pad, P51 Pad, P52 Pad, P53 Pad, P56 Pad, P6 Pad, P7 Pad, P8 Pad, P9 Pad, Q1 AUIPS2041LTR, Q2 AUIPS2041LTR, U1 LIS2DW12TR, U2 MPX4_MAP, U3 MCP6002-xSN, U4 LPS25HB, U5 L6205PD

Commit message: update schem.
Parts:
- removed J3: MiniFit, hellen-one-common:Molex-39301020, symbol Connector_Generic:Conn_01x02
- removed J6: ETB, hellen-one-common:PinHeader_1x08_P2.54mm_Vertical, symbol Connector_Generic:Conn_01x08
- removed P17: Pad, hellen-one-common:PAD-TH, symbol hellen-one-common:Pad
- D35, D36: footprint Diode_SMD:D_SOD-123 -> hellen-one-common:SOD-123
- Q1, Q2: footprint Package_TO_SOT_SMD:SOT-223 -> hellen-one-common:SOT-223
- R28, R29: footprint Resistor_SMD:R_0402_1005Metric -> hellen-one-common:R0603; LCSC C60489 -> C25804
Connections:
- net 4K: no longer M12.E5 (LSU_H+), P2.38 (1W)
- net GND: now also R28.2, R29.2; no longer R28.1, R29.1
- net GNDA: now also P2.3 (1L), P2.34 (1K); no longer P2.33 (1H), P2.68 (1G)
- net IDLE: now also R29.1; no longer R29.2
- net IN_PPS: now also P2.2 (1F); no longer P2.34 (1K)
- net IN_TEMP_OR_PPS2: now also P2.32 (1E); no longer P2.69 (1J)
- net IN_TPS: now also P2.33 (1H); no longer P2.70 (1M)
- net IN_TPS2: now also P2.68 (1G); no longer P2.3 (1L)
- net OUT_ETB+: now also P2.69 (1J)
- net OUT_ETB-: now also P2.70 (1M)
- net VVT: now also R28.1; no longer R28.2
- net 1C: now reaches P19.1 (Pin_1), P2.1 (1C)
- net 1Q: now reaches P16.1 (Pin_1), P2.36 (1Q)
- net 1R: now reaches P2.5 (1R), P3.1 (Pin_1)
- net 1D: now reaches P2.67 (1D), R43.2
- net 4L renamed 1X
- new net WBO_H-: M12.E5 (LSU_H+), P2.38 (1W)
Other:
- moved on the sheet: F2, F3, P10, P15, P16, P19, P3, P52, P53, P8, P9, R12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

Commit message: update schematics with 8-5353015-1
Parts:
- removed P16, P3: Pad, hellen-one-common:PAD-TH, symbol hellen-one-common:Pad
- added J3: MiniFit, hellen-one-common:Molex-39301020, symbol Connector_Generic:Conn_01x02
- added unit 5 of P2
- P2: value 1123794-2 -> 8-5353015-1; footprint hellen-one-common:1123794-2 -> NB2:8-5353015-1; symbol 1123794-2:1123794-2 -> 8-5353015-1:8-5353015-1
Connections:
- net +12V_PERM: now also P2.84 (4AG); no longer P2.65 (4AG)
- net +12V_RAW: now also P2.106 (2P), P2.115 (4D), P2.55 (5W), P2.98 (5V); no longer P2.78 (2P), P2.87 (4D)
- net +5VA: now also P2.116 (4L), P2.53 (5R), P2.97 (5P); no longer P2.35 (1N), P2.4 (1O), P2.88 (4L)
- net 2C: now also P2.17 (2C); no longer P2.8 (2C)
- net 2E: now also P2.59 (2E); no longer P2.40 (2E)
- net 2F: now also P2.18 (2F); no longer P2.9 (2F)
- net 2H: now also P2.60 (2H); no longer P2.41 (2H)
- net 2I: now also P2.19 (2I); no longer P2.10 (2I)
- net 2N: now also P2.62 (2N); no longer P2.43 (2N)
- net 3C: now also P2.22 (3C); no longer P2.13 (3C)
- net 3D: now also P2.108 (3D); no longer P2.80 (3D)
- net 3H: now also P2.66 (3H); no longer P2.47 (3H)
- net 3J: now also P2.109 (3J); no longer P2.81 (3J)
- net 3Q: now also P2.69 (3Q); no longer P2.50 (3Q)
- net 3S: now also P2.70 (3S); no longer P2.51 (3S)
- net 3U: now also P2.112 (3U); no longer P2.84 (3U)
- net 3W: now also P2.28 (3W); no longer P2.19 (3W)
- net 3X: now also P2.113 (3X); no longer P2.85 (3X)
- net 3Z: now also P2.29 (3Z); no longer P2.20 (3Z)
- net 4AB: now also P2.37 (4AB); no longer P2.28 (4AB)
- net 4AC: now also P2.121 (4AC); no longer P2.93 (4AC)
- net 4AD: now also P2.83 (4AD); no longer P2.64 (4AD)
- net 4AE: now also P2.38 (4AE); no longer P2.29 (4AE)
- net 4AF: now also P2.122 (4AF); no longer P2.94 (4AF)
- net 4E: now also P2.74 (4E); no longer P2.55 (4E)
- net 4K: now also P2.33 (4K); no longer P2.24 (4K)
- net 4M: now also P2.77 (4M); no longer P2.58 (4M)
- net 4S: now also P2.79 (4S); no longer P2.60 (4S)
- net 4Z: now also P2.120 (4Z); no longer P2.92 (4Z)
- net GND: now also P2.107 (3A), P2.114 (4A), P2.64 (3B), P2.14 (5X), P2.94 (5H); no longer P2.45 (3B), P2.66 (1A), P2.79 (3A), P2.86 (4A)
- net GNDA: now also P2.117 (4O), P2.12 (5S), P2.54 (5T); no longer P2.3 (1L), P2.34 (1K), P2.89 (4O)
- net IN_AC_PRESSURE: now also P2.31 (4F); no longer P2.22 (4F)
- net IN_AFR: now also P2.25 (3L); no longer P2.16 (3L)
- net IN_BRAKE: now also P2.73 (4B); no longer P2.54 (4B)
- net IN_CAM: now also P2.71 (3V); no longer P2.52 (3V)
- net IN_CLT: now also P2.78 (4P); no longer P2.59 (4P)
- net IN_CLUTCH: now also P2.32 (4I); no longer P2.23 (4I)
- net IN_CRANK: now also P2.72 (3Y); no longer P2.53 (3Y)
- net IN_DIGITAL: now also P2.50 (5I); no longer P2.31 (1B)
- net IN_IAT: now also P2.34 (4N); no longer P2.25 (4N)
- net IN_MAF: now also P2.81 (4X); no longer P2.62 (4X)
- net IN_MAP: now also P2.119 (4U); no longer P2.91 (4U)
- net IN_NEUTRAL: now also P2.75 (4H); no longer P2.56 (4H)
- net IN_O2S2: now also P2.36 (4W); no longer P2.27 (4W)
- net IN_O2S3: now also P2.82 (4AA); no longer P2.63 (4AA)
- net IN_PPS: now also P2.96 (5M); no longer P2.2 (1F)
- net IN_SENS2: now also P2.67 (3K); no longer P2.48 (3K)
- net IN_STEERING: now also P2.30 (4C); no longer P2.21 (4C)
- net IN_TEMP_OR_PPS2: now also P2.51 (5L); no longer P2.32 (1E)
- net IN_TPS: now also P2.80 (4V), P2.11 (5O); no longer P2.33 (1H), P2.61 (4V)
- net IN_TPS2: now also P2.52 (5N); no longer P2.68 (1G)
- net IN_VSS: now also P2.27 (3T); no longer P2.18 (3T)
- net IN_VTCS: now also P2.76 (4J); no longer P2.57 (4J)
- net OUT_AC_RELAY: now also P2.61 (2K); no longer P2.42 (2K)
- net OUT_ALTERNATOR: now also P2.110 (3M); no longer P2.82 (3M)
- net OUT_CHECK_ENGINE: now also P2.21 (2R); no longer P2.12 (2R)
- net OUT_ECF_RELAY: now also P2.58 (2B); no longer P2.39 (2B)
- net OUT_ETB+: now also J3.2 (Pin_2); no longer P2.69 (1J)
- net OUT_ETB-: now also J3.1 (Pin_1); no longer P2.70 (1M)
- net OUT_IDLE: now also P2.63 (2Q); no longer P2.44 (2Q)
- net OUT_IGN1: now also P2.23 (3F); no longer P2.14 (3F)
- net OUT_IGN2: now also P2.24 (3I); no longer P2.15 (3I)
- net OUT_IGN3: now also P2.20 (2O); no longer P2.11 (2O)
- net OUT_IGN4: now also P2.68 (3N); no longer P2.49 (3N)
- net OUT_INJ1: now also P2.101 (2A); no longer P2.73 (2A)
- net OUT_INJ2: now also P2.102 (2D); no longer P2.74 (2D)
- net OUT_INJ3: now also P2.103 (2G); no longer P2.75 (2G)
- net OUT_INJ4: now also P2.104 (2J); no longer P2.76 (2J)
- net OUT_PUMP_RELAY: now also P2.105 (2M); no longer P2.77 (2M)
- net OUT_TACH: now also P2.26 (3O); no longer P2.17 (3O)
- net OUT_VVT: now also P2.118 (4R); no longer P2.90 (4R)
- net WBO_H-: now also P2.57 (5AD); no longer P2.38 (1W)
- net WBO_Ip: now also P2.100 (5AC); no longer P2.72 (1V)
- net WBO_R_Trim: now also P2.15 (5AB); no longer P2.6 (1U)
- net WBO_Vs: now also P2.56 (5AA); no longer P2.37 (1T)
- net WBO_Vs/Ip: now also P2.99 (5Z); no longer P2.71 (1S)
- net at P50.1 (Pin_1): now also P2.39 (4AH); no longer P2.30 (4AH)
- net at R27.1: now also P2.65 (3E); no longer P2.46 (3E)
- net at R18.2: now also P2.111 (3P); no longer P2.83 (3P)
- net 1C: no longer names the net of P2.1 (1C)
- net 1C: no longer P19.1 (Pin_1)
- net 1D renamed 5K
- net 5K: now also P2.95 (5K); no longer P2.67 (1D)
- removed net 1Q: P2.36 (1Q)
- net 1R: no longer names the net of P2.5 (1R)
- net 1X: no longer names the net of P2.7 (1X)
- net 1X: no longer F2.1
- new net 5AE: F2.1, P2.16 (5AE)
- new net 5J: P19.1 (Pin_1), P2.10 (5J)
- no-connect marks 52 -> 59
Other:
- moved on the sheet: D1, D10, D11, D12, D13, D14, D15, D16, D17, D18, D19, D2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

Commit message: update schematics & pcb
Parts:
- removed D25, D28, D32: B5819W, hellen-one-common:SOD-123, symbol hellen-one-common:1N4148WS
- removed P20: Pad, hellen-one-common:PAD-TH, symbol hellen-one-common:Pad
- added D25, D28: LED-BLUE-0603, hellen-one-common:LED-0603, symbol hellen-one-common:LED_0603
- added F4, F5: Fuse-Pad-Pad, hellen-one-common:PAD-1206-PAD, symbol hellen-one-common:Fuse-Pad-Pad
- added P16, P17, P21, P3: Pad, hellen-one-common:PAD-TH, symbol hellen-one-common:Pad
- added R30, R33, R34: Jumper-Pad-Pad, hellen-one-common:PAD-0805-PAD, symbol hellen-one-common:Jumper-Pad-Pad
- renumbered R46 to R1, R21 to R10, R22 to R11, R7 to R20, R10 to R21, R11 to R22, R9 to R35, R1 to R36, R8 to R5, R5 to R55, R20 to R7, R42 to R8, R36 to R9
Connections:
- net IN_PRESSURE is gone; now on net IN_AC_PRESSURE: R22.1
- net IO8 is gone; now on net IO12: M3.E13 (OUT_IO12), P5.1 (Pin_1)
- net OUT_LOW1 is gone; now on net OUT_ECF_RELAY: M5.S8 (OUT_LOW1)
- net +12V_RAW: now also F4.2, F5.2; no longer P2.55 (5W), P2.98 (5V)
- net +5VA: now also P2.12 (5S); no longer P2.97 (5P)
- net GNDA: now also P2.13 (5U); no longer P2.12 (5S)
- net IN_IAT: now also R33.1, R34.1; no longer P2.34 (4N)
- net IN_PPS: now also P2.97 (5P); no longer P2.96 (5M)
- net IO12: no longer M3.E23 (OUT_IO4), P4.1 (Pin_1)
- net O2H2: now also M3.E12 (OUT_IO2); no longer M3.E11 (OUT_IO9)
- net OUT_IDLE: now also Q2.4 (D)
- net OUT_IGN2: now also D25.1 (A); no longer D4.1 (A)
- net OUT_IGN3: now also D28.1 (A)
- net OUT_IGN4: now also D4.1 (A)
- net OUT_INJ8_BOOST: now also D31.2 (A), M5.W11 (OUT_INJ8)
- net OUT_VVT: now also Q1.4 (D), R30.1; no longer P2.118 (4R)
- net at R36.6: now also D28.2 (K)
- net at R36.7: now also D25.2 (K)
- net 1A: now reaches P2.85 (1A)
- net 1A: now also P21.1 (Pin_1)
- net 1D: now reaches P2.86 (1D)
- net 1D: now also P17.1 (Pin_1)
- net 1G: now reaches P2.87 (1G)
- net 1G: now also P16.1 (Pin_1)
- net 1J: now reaches P2.88 (1J)
- net 1J: now also P3.1 (Pin_1)
- net AC_FAN_RELAY: no longer names the net of M5.W29 (LOW2)
- net AC_FAN_RELAY: no longer M3.E12 (OUT_IO2)
- net BOOST renamed INJ6
- net IN_TEMP_OR_PPS2: no longer names the net of P2.51 (5L)
- net IN_TEMP_OR_PPS2: no longer M1.S18 (IN_AUX2)
- net LOW1 renamed ECF_RELAY
- net OUT_AC_FAN_RELAY: no longer names the net of M5.W1 (OUT_LOW2)
- net PP1 renamed ALTERN
- net PP2 renamed TACH
- net TEMP renamed PPS2
- net VICS renamed INJ8_BOOST
- new net: F5.1, P2.55 (5W)
- new net: F4.1, P2.98 (5V)
- new net: P2.118 (4R), R30.2, R33.2
- new net: P2.34 (4N), R34.2
- new net IN_PPS2: M1.S18 (IN_AUX2), P2.96 (5M)
- new net IO4: M3.E23 (OUT_IO4), P4.1 (Pin_1)
- no-connect marks 59 -> 80
Other:
- note added: "3L (Not OEM)"
- note added: "3Z (Not OEM)"
- note added: "4K (Not OEM)"
- note added: "4U (Not OEM)"
- note added: "IN_TEMP"
- note added: "MSM"
- note added: "Miata 2002"
- note added: "Miata 2003"
- note added: "OUT_AC_FAN_RELAY"
- note removed: "Not OEM"
- note removed: "OUT_INJ8_BOOST"
- moved on the sheet: C21, D31, D35, D36, Q1, Q2, R28, R29

Commit message: update
Parts:
- added F6: Fuse-Pad-Pad, hellen-one-common:PAD-1206-PAD, symbol hellen-one-common:Fuse-Pad-Pad
- added R37: Jumper-Pad-Pad, hellen-one-common:PAD-0805-PAD, symbol hellen-one-common:Jumper-Pad-Pad
- M3: value Module-mcu144-0.5 -> Module-mcu144-0.6; footprint hellen-one-mcu-0.5:mcu -> hellen-one-mcu-0.6:mcu; symbol hellen-one-mcu-0.5:Module-mcu-0.5 -> hellen-one-mcu-0.6:Module-mcu-0.6
Connections:
- net +12V_RAW: no longer P2.115 (4D)
- net 4AF: now also F6.2
- net OUT_INJ8_BOOST: now also R37.1
- new net: F6.1, P2.115 (4D), R37.2

Commit message: update rev.E
Parts:
- removed P14, P22, P28, P38, P44: Pad, hellen-one-common:PAD-TH, symbol hellen-one-common:Pad
- added P20: Pad, hellen-one-common:PAD-TH, symbol hellen-one-common:Pad
- C21: LCSC C14663 -> (none); MyComment (none) -> DNP
- R23: value 1k -> 0; LCSC C21190 -> C21189
Connections:
- net +5VA: now also P2.51 (5L)
- net IN_D4: now also P2.8 (5C)
- net IN_RES3: now also P2.48 (5B)
- net IN_SENS3: now also P2.93 (5D)
- net OUT_HIGH1: now also P2.9 (5F)
- net OUT_SOLENOID_B2: now also P2.49 (5E)
- net IN_MAP1: now reaches P2.92 (5A)
- net IN_MAP1: now also M1.S11 (IN_MAP1), R4.1
- removed net IN_MAF: M1.S11 (IN_MAP1), P2.81 (4X), R4.1
- net IN_MAP renamed IN_MAP2
- net MAF renamed MAP1
- new net: P2.81 (4X), P20.1 (Pin_1)
- no-connect marks 80 -> 73
Other:
- note added: "IN_MAF"
- note added: "https://www.youtube.com/watch?v=KLWQtNRfnZc"

Commit message: mcu-176
Parts:
- M3: value Module-mcu144-0.6 -> Module-mcu-0.6
Changed lines of the file:
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@@
       (effects (font (size 1.27 1.27)) (justify left))
     )
-    (property "Value" "Module-mcu144-0.6" (id 1) (at 418.4651 206.0078 0)
+    (property "Value" "Module-mcu-0.6" (id 1) (at 418.4651 206.0078 0)
       (effects (font (size 1.27 1.27)) (justify left))
     )
@@
       (effects (font (size 1.27 1.27)) (justify right))
     )
-    (property "Value" "Module-mcu144-0.6" (id 1) (at 418.4651 67.5778 0)
+    (property "Value" "Module-mcu-0.6" (id 1) (at 418.4651 67.5778 0)
       (effects (font (size 1.27 1.27)) (justify right))
     )
@@
     (in_bom yes) (on_board yes)
     (property "Reference" "M3" (id 0) (at 445.9605 65.2738 0))
-    (property "Value" "Module-mcu144-0.6" (id 1) (at 451.0405 67.5725 0))
+    (property "Value" "Module-mcu-0.6" (id 1) (at 451.0405 67.5725 0))
     (property "Footprint" "hellen-one-mcu-0.6:mcu" (id 2) (at 435.61 68.58 0)
       (effects (font (size 1.27 1.27)) hide)
@@
     (in_bom yes) (on_board yes) (fields_autoplaced)
     (property "Reference" "M3" (id 0) (at 473.71 215.1338 0))
-    (property "Value" "Module-mcu144-0.6" (id 1) (at 473.71 217.4325 0))
+    (property "Value" "Module-mcu-0.6" (id 1) (at 473.71 217.4325 0))
     (property "Footprint" "hellen-one-mcu-0.6:mcu" (id 2) (at 455.93 218.44 0)
       (effects (font (size 1.27 1.27)) hide)
@@
     )
     (path "/a6bf355d-1d5f-4e79-8e3f-45e3bddf3ceb"
-      (reference "M3") (unit 1) (value "Module-mcu144-0.6") (footprint "hellen-one-mcu-0.6:mcu")
+      (reference "M3") (unit 1) (value "Module-mcu-0.6") (footprint "hellen-one-mcu-0.6:mcu")
     )
     (path "/915d735b-9683-4d94-8b0d-1fa27ebac489"
-      (reference "M3") (unit 2) (value "Module-mcu144-0.6") (footprint "hellen-one-mcu-0.6:mcu")
+      (reference "M3") (unit 2) (value "Module-mcu-0.6") (footprint "hellen-one-mcu-0.6:mcu")
     )
     (path "/5f1c7f30-e456-4e5e-847b-c87579bb1a4c"
-      (reference "M3") (unit 3) (value "Module-mcu144-0.6") (footprint "hellen-one-mcu-0.6:mcu")
+      (reference "M3") (unit 3) (value "Module-mcu-0.6") (footprint "hellen-one-mcu-0.6:mcu")
     )
     (path "/a7d95f89-5755-415c-ab05-3cba0bcc1e6a"
-      (reference "M3") (unit 4) (value "Module-mcu144-0.6") (footprint "hellen-one-mcu-0.6:mcu")
+      (reference "M3") (unit 4) (value "Module-mcu-0.6") (footprint "hellen-one-mcu-0.6:mcu")
     )
     (path "/46c92d79-ab77-4cea-933a-f95fdcee2757"

Commit message: https://github.com/rusefi/hellen-NB2-issues/issues/34
Connections:
- net OUT_IDLE: no longer Q2.4 (D)
- net OUT_VVT: no longer Q1.4 (D)
Changed lines of the file:
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@@
   (title_block
     (title "Hellen72 NB2")
-    (date "2022-03-05")
-    (rev "E")
+    (date "2022-03-28")
+    (rev "F")
     (company "rusEFI")
     (comment 7 "http://rusefi.com/s/hellenNB2")
@@
   (symbol (lib_id "Power_Management:AUIPS2041L") (at 273.05 53.34 0) (mirror y) (unit 1)
     (in_bom yes) (on_board yes)
-    (property "Reference" "Q2" (id 0) (at 267.97 58.42 0)
+    (property "Reference" "Q2" (id 0) (at 278.13 58.42 0)
       (effects (font (size 1.27 1.27)) (justify left))
     )
@@
     (pin "2")
     (pin "3")
-    (pin "4")
   )
   (symbol (lib_id "hellen-one-knock-0.1:Module-knock-0.1") (at 218.44 275.59 0) (unit 1)
@@
   (symbol (lib_name "AUIPS2041L_1") (lib_id "Power_Management:AUIPS2041L") (at 245.11 55.88 0) (mirror y) (unit 1)
     (in_bom yes) (on_board yes)
-    (property "Reference" "Q1" (id 0) (at 238.76 58.42 0)
+    (property "Reference" "Q1" (id 0) (at 251.46 58.42 0)
       (effects (font (size 1.27 1.27)) (justify left))
     )
-    (property "Value" "AUIPS2041LTR" (id 1) (at 242.57 60.96 0)
+    (property "Value" "AUIPS2041LTR" (id 1) (at 247.65 60.96 0)
       (effects (font (size 1.27 1.27)) (justify left))
     )
@@
     (pin "2")
     (pin "3")
-    (pin "4")
   )
   (symbol (lib_id "hellen-one-common:Jumper-Pad-Pad") (at 127 30.48 0) (mirror y) (unit 1)
